File: Eagle/ECHO.brd (EAGLE design)
At the start: 29.1 x 44.9 mm, 13 parts, among them IC1 AT24C, T1 IRLML6402

Commit message: finished pcb layout
Parts:
- moved R2 2.65 mm to (29.2, 17.5), turned to 90 degrees
- moved MICROPHONE 0.76 mm to (31.8, 13.5)
Connections:
- removed net N$4: MICROPHONE.2, R2.1
- new net N$3: MICROPHONE.1, R2.1
- net GND: now also MICROPHONE.2; no longer MICROPHONE.3
- net VCC: now also MICROPHONE.3; no longer MICROPHONE.1
Routing:
- net VCC: track 62.3 -> 68.3 mm
- net N$4: track 4.42 -> 0.00 mm
- net N$3: track 0.00 -> 3.21 mm
- net GND: track 96.1 -> 93.2 mm
- net AUD: track 14.4 -> 12.1 mm
Other:
- board text added: "1"
- board text added: "100nF"
- board text added: "1M"
- board text added: "2"
- board text added: "25"
- board text added: "26"
- board text added: "3K16"
- board text added: "47nF"
- board text added: "4K87"
- board text added: "AUD"
- board text added: "C1"
- board text added: "C2"
- board text added: "CSE 477: Team 4 Project: Echo Version: 1.0"
- board text added: "CTS"
- board text added: "DTR"
- board text added: "EEPROM"
- board text added: "GND"
- board text added: "J1"
- board text added: "R1"
- board text added: "R2"
- board text added: "R3"
- board text added: "RESET"
- board text added: "RXI"
- board text added: "T1"
- board text added: "TXO"
- board text added: "VCC"

Commit message: before revamp of envelope
Parts:
- removed IC1: AT24C, atmel:SOIC8
- added SRAM: AT24CP, atmel:DIL08
- moved C2 13.2 mm to (21.6, 28.2)
- moved JP2 13.2 mm to (1.52, 23.9)
- moved MICROPHONE 13.2 mm to (23.4, 3.30)
- moved R1 13.2 mm to (10.7, 7.37)
- moved R2 13.2 mm to (20.8, 7.37)
- moved RESET_BUTTON 13.2 mm to (22.9, 15.5)
- moved C1 13.2 mm to (5.08, 7.37)
- moved FTDI_HEADER 13.2 mm to (2.29, 2.79)
- moved R3 13.2 mm to (15.7, 8.13)
- moved T1 13.2 mm to (16.5, 7.62)
- moved J1 13.2 mm to (13.0, 27.7)
Connections:
- removed net I2C_SCL: IC1.6, J1.1
- removed net I2C_SDA: IC1.5, J1.3
- new net SPI_CS: J1.7, SRAM.1
- new net SPI_MISO: J1.12, SRAM.2
- new net SPI_MOSI: J1.10, SRAM.5
- new net SPI_SCK: J1.8, SRAM.6
- net GND: now also SRAM.4, SRAM.7; no longer IC1.1, IC1.2, IC1.3, IC1.4, IC1.7
- net VBUS: now also C2.1, SRAM.8
- net VCC: no longer C2.1, IC1.8
Routing:
- net VCC: track 68.3 -> 40.0 mm
- net SPI_MISO: track 0.00 -> 23.8 mm
- net VBUS: track 7.47 -> 30.4 mm
- net SPI_CS: track 0.00 -> 14.0 mm
- net GND: track 93.2 -> 80.5 mm
- net I2C_SCL: track 12.0 -> 0.00 mm
- net SPI_SCK: track 0.00 -> 11.3 mm
- net I2C_SDA: track 8.61 -> 0.00 mm
- net SPI_MOSI: track 0.00 -> 7.91 mm
