File: Eagle/ECHO.sch (EAGLE design)
At the start: 13 parts, among them IC1 AT24C, T1 IRLML6402

Commit message: finished pcb layout
Connections:
- removed net N$4: MICROPHONE.2, R2.1
- new net N$3: MICROPHONE.1, R2.1
- net GND: now also MICROPHONE.2; no longer MICROPHONE.3
- net VCC: now also MICROPHONE.3; no longer MICROPHONE.1
Other:
- moved on the sheet: R2, R3
Changed lines of the file:
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@@
 <grid distance="0.1" unitdist="inch" unit="inch" style="lines" multiple="1" display="no" altdistance="0.01" altunitdist="inch" altunit="inch"/>
 <layers>
-<layer number="1" name="Top" color="4" fill="1" visible="yes" active="no"/>
-<layer number="16" name="Bottom" color="1" fill="1" visible="yes" active="no"/>
-<layer number="17" name="Pads" color="2" fill="1" visible="yes" active="no"/>
-<layer number="18" name="Vias" color="2" fill="1" visible="yes" active="no"/>
-<layer number="19" name="Unrouted" color="6" fill="1" visible="yes" active="no"/>
-<layer number="20" name="Dimension" color="15" fill="1" visible="yes" active="no"/>
-<layer number="21" name="tPlace" color="7" fill="1" visible="yes" active="no"/>
-<layer number="22" name="bPlace" color="7" fill="1" visible="yes" active="no"/>
-<layer number="23" name="tOrigins" color="15" fill="1" visible="yes" active="no"/>
-<layer number="24" name="bOrigins" color="15" fill="1" visible="yes" active="no"/>
-<layer number="25" name="tNames" color="7" fill="1" visible="yes" active="no"/>
-<layer number="26" name="bNames" color="7" fill="1" visible="yes" active="no"/>
-<layer number="27" name="tValues" color="7" fill="1" visible="yes" active="no"/>
-<layer number="28" name="bValues" color="7" fill="1" visible="yes" active="no"/>
+<layer number="1" name="Top" color="4" fill="1" visible="no" active="no"/>
+<layer number="16" name="Bottom" color="1" fill="1" visible="no" active="no"/>
+<layer number="17" name="Pads" color="2" fill="1" visible="no" active="no"/>
+<layer number="18" name="Vias" color="2" fill="1" visible="no" active="no"/>
+<layer number="19" name="Unrouted" color="6" fill="1" visible="no" active="no"/>
+<layer number="20" name="Dimension" color="15" fill="1" visible="no" active="no"/>
+<layer number="21" name="tPlace" color="7" fill="1" visible="no" active="no"/>
+<layer number="22" name="bPlace" color="7" fill="1" visible="no" active="no"/>
+<layer number="23" name="tOrigins" color="15" fill="1" visible="no" active="no"/>
+<layer number="24" name="bOrigins" color="15" fill="1" visible="no" active="no"/>
+<layer number="25" name="tNames" color="7" fill="1" visible="no" active="no"/>
+<layer number="26" name="bNames" color="7" fill="1" visible="no" active="no"/>
+<layer number="27" name="tValues" color="7" fill="1" visible="no" active="no"/>
+<layer number="28" name="bValues" color="7" fill="1" visible="no" active="no"/>
 <layer number="29" name="tStop" color="7" fill="3" visible="no" active="no"/>
 <layer number="30" name="bStop" color="7" fill="6" visible="no" active="no"/>
@@
 <layer number="35" name="tGlue" color="7" fill="4" visible="no" active="no"/>
 <layer number="36" name="bGlue" color="7" fill="5" visible="no" active="no"/>
-<layer number="37" name="tTest" color="7" fill="1" visible="yes" active="no"/>
-<layer number="38" name="bTest" color="7" fill="1" visible="yes" active="no"/>
+<layer number="37" name="tTest" color="7" fill="1" visible="no" active="no"/>
+<layer number="38" name="bTest" color="7" fill="1" visible="no" active="no"/>
 <layer number="39" name="tKeepout" color="4" fill="11" visible="no" active="no"/>
 <layer number="40" name="bKeepout" color="1" fill="11" visible="no" active="no"/>
@@
 <layer number="44" name="Drills" color="7" fill="1" visible="no" active="no"/>
 <layer number="45" name="Holes" color="7" fill="1" visible="no" active="no"/>
-<layer number="46" name="Milling" color="3" fill="1" visible="yes" active="no"/>
-<layer number="47" name="Measures" color="7" fill="1" visible="yes" active="no"/>
-<layer number="48" name="Document" color="7" fill="1" visible="yes" active="no"/>
-<layer number="49" name="Reference" color="7" fill="1" visible="yes" active="no"/>
-<layer number="50" name="dxf" color="7" fill="1" visible="yes" active="no"/>
-<layer number="51" name="tDocu" color="7" fill="1" visible="yes" active="no"/>
-<layer number="52" name="bDocu" color="7" fill="1" visible="yes" active="no"/>
-<layer number="53" name="tGND_GNDA" color="7" fill="9" visible="yes" active="no"/>
-<layer number="54" name="bGND_GNDA" color="1" fill="9" visible="yes" active="no"/>
-<layer number="56" name="wert" color="7" fill="1" visible="yes" active="no"/>
-<layer number="57" name="tCAD" color="7" fill="1" visible="yes" active="no"/>
+<layer number="46" name="Milling" color="3" fill="1" visible="no" active="no"/>
+<layer number="47" name="Measures" color="7" fill="1" visible="no" active="no"/>
+<layer number="48" name="Document" color="7" fill="1" visible="no" active="no"/>
+<layer number="49" name="Reference" color="7" fill="1" visible="no" active="no"/>
+<layer number="50" name="dxf" color="7" fill="1" visible="no" active="no"/>
+<layer number="51" name="tDocu" color="7" fill="1" visible="no" active="no"/>
+<layer number="52" name="bDocu" color="7" fill="1" visible="no" active="no"/>
+<layer number="53" name="tGND_GNDA" color="7" fill="9" visible="no" active="no"/>
+<layer number="54" name="bGND_GNDA" color="1" fill="9" visible="no" active="no"/>
+<layer number="56" name="wert" color="7" fill="1" visible="no" active="no"/>
+<layer number="57" name="tCAD" color="7" fill="1" visible="no" active="no"/>
 <layer number="91" name="Nets" color="2" fill="1" visible="yes" active="yes"/>
 <layer number="92" name="Busses" color="1" fill="1" visible="yes" active="yes"/>
@@
 <instance part="GND3" gate="1" x="99.06" y="101.6"/>
 <instance part="MICROPHONE" gate="A" x="50.8" y="78.74"/>
-<instance part="R2" gate="G$1" x="20.32" y="78.74" rot="R180"/>
-<instance part="R3" gate="G$1" x="12.7" y="66.04" rot="R90"/>
-<instance part="GND4" gate="1" x="12.7" y="48.26"/>
+<instance part="R2" gate="G$1" x="22.86" y="81.28" rot="R180"/>
+<instance part="R3" gate="G$1" x="15.24" y="68.58" rot="R90"/>
+<instance part="GND4" gate="1" x="15.24" y="50.8"/>
 <instance part="GND5" gate="1" x="76.2" y="40.64"/>
 <instance part="C2" gate="G$1" x="81.28" y="60.96"/>
@@
 </segment>
 <segment>
-<pinref part="MICROPHONE" gate="A" pin="3"/>
-<wire x1="48.26" y1="76.2" x2="33.02" y2="76.2" width="0.1524" layer="91"/>
-<label x="33.02" y="76.2" size="1.778" layer="95"/>
-</segment>
-<segment>
 <pinref part="R3" gate="G$1" pin="1"/>
-<wire x1="12.7" y1="60.96" x2="12.7" y2="50.8" width="0.1524" layer="91"/>
+<wire x1="15.24" y1="63.5" x2="15.24" y2="53.34" width="0.1524" layer="91"/>
 <pinref part="GND4" gate="1" pin="GND"/>
 </segment>
@@
 <pinref part="IC1" gate="G$1" pin="A0"/>
 </segment>
+<segment>
+<pinref part="MICROPHONE" gate="A" pin="2"/>
+<wire x1="48.26" y1="78.74" x2="35.56" y2="78.74" width="0.1524" layer="91"/>
+<label x="35.56" y="78.74" size="1.778" layer="95"/>
+</segment>
 </net>
 <net name="VCC" class="0">
@@
 <wire x1="160.02" y1="93.98" x2="147.32" y2="93.98" width="0.1524" layer="91"/>
 <label x="149.86" y="93.98" size="1.778" layer="95"/>
-</segment>
-<segment>
-<pinref part="MICROPHONE" gate="A" pin="1"/>
-<wire x1="48.26" y1="81.28" x2="33.02" y2="81.28" width="0.1524" layer="91"/>
-<label x="33.02" y="81.28" size="1.778" layer="95"/>
 </segment>
 <segment>
@@
 <junction x="81.28" y="68.58"/>
 <pinref part="IC1" gate="G$1" pin="VCC"/>
+</segment>
+<segment>
+<pinref part="MICROPHONE" gate="A" pin="3"/>
+<wire x1="48.26" y1="76.2" x2="35.56" y2="76.2" width="0.1524" layer="91"/>
+<label x="35.56" y="76.2" size="1.778" layer="95"/>
 </segment>
 </net>
@@
 <segment>
 <pinref part="R2" gate="G$1" pin="2"/>
-<wire x1="15.24" y1="78.74" x2="12.7" y2="78.74" width="0.1524" layer="91"/>
+<wire x1="17.78" y1="81.28" x2="15.24" y2="81.28" width="0.1524" layer="91"/>
 <pinref part="R3" gate="G$1" pin="2"/>
-<wire x1="12.7" y1="78.74" x2="12.7" y2="71.12" width="0.1524" layer="91"/>
-<wire x1="12.7" y1="78.74" x2="12.7" y2="88.9" width="0.1524" layer="91"/>
-<wire x1="12.7" y1="88.9" x2="15.24" y2="91.44" width="0.1524" layer="91"/>
-<junction x="12.7" y="78.74"/>
-<label x="15.24" y="91.44" size="1.778" layer="95"/>
+<wire x1="15.24" y1="81.28" x2="15.24" y2="73.66" width="0.1524" layer="91"/>
+<wire x1="15.24" y1="81.28" x2="15.24" y2="91.44" width="0.1524" layer="91"/>
+<wire x1="15.24" y1="91.44" x2="17.78" y2="93.98" width="0.1524" layer="91"/>
+<junction x="15.24" y="81.28"/>
+<label x="17.78" y="93.98" size="1.778" layer="95"/>
 </segment>
 <segment>
@@
 </segment>
 </net>
-<net name="N$4" class="0">
-<segment>
-<pinref part="MICROPHONE" gate="A" pin="2"/>
-<pinref part="R2" gate="G$1" pin="1"/>
-<wire x1="48.26" y1="78.74" x2="25.4" y2="78.74" width="0.1524" layer="91"/>
-</segment>
-</net>
 <net name="I2C_SCL" class="0">
 <segment>
@@
 </segment>
 </net>
+<net name="N$3" class="0">
+<segment>
+<pinref part="MICROPHONE" gate="A" pin="1"/>
+<pinref part="R2" gate="G$1" pin="1"/>
+<wire x1="48.26" y1="81.28" x2="27.94" y2="81.28" width="0.1524" layer="91"/>
+</segment>
+</net>

Commit message: before revamp of envelope
Parts:
- removed IC1: AT24C, atmel:AT24C
- added SRAM: AT24CP, atmel:AT24CP
Connections:
- removed net I2C_SCL: IC1.SCL, J1.1
- removed net I2C_SDA: IC1.SDA, J1.3
- new net SPI_CS: J1.7, SRAM.A0
- new net SPI_MISO: J1.12, SRAM.A1
- new net SPI_MOSI: J1.10, SRAM.SDA
- new net SPI_SCK: J1.8, SRAM.SCL
- net GND: now also SRAM.GND, SRAM.WP; no longer IC1.A0, IC1.A1, IC1.A2, IC1.GND, IC1.WP
- net VBUS: now also C2.1, SRAM.VCC
- net VCC: no longer C2.1, IC1.VCC
